File: Hardware/PI-CNC.sch (KiCad schematic (older format))
At the start: 18 parts, among them J3 40HAT, J6 CONN_02X02, J9 CONN_01X02, Q1 DMG2305UX, Q2 DMMT5401, U2 CAT24C32

Commit message: Main Parts on schematic and board.
Parts:
- added A1, A2, A3, A4: Pololu_Breakout_A4988, Module:Pololu_Breakout-16_15.2x20.3mm, symbol Driver_Motor:Pololu_Breakout_A4988
- added C1: C, Capacitor_SMD:C_1210_3225Metric, symbol Device:C
- added U1: TPS54360DDA, Package_SO:TI_SO-PowerPAD-8_ThermalVias, symbol Regulator_Switching:TPS54360DDA
- added U3: DS1339+, Package_SO:MSOP-8_3x3mm_P0.65mm, symbol Timer_RTC:DS1307+
- added U4: CP2102N-A01-GQFN28, Package_DFN_QFN:QFN-28-1EP_5x5mm_P0.5mm_EP3.35x3.35mm, symbol Interface_USB:CP2102N-A01-GQFN28
- added U5: ATmega2560-16AU, Package_QFP:TQFP-100_14x14mm_P0.5mm, symbol MCU_Microchip_ATmega:ATmega2560-16AU
Connections:
- net GND: now also C1.2
- net P5V_HAT: no longer J3.2 (P5V), J3.4 (P5V)
- net Console_RX: now reaches J3.10 (BCM15)
- net LED_white: now reaches J3.12 (BCM18)
- net LED_red: now reaches J3.16 (BCM23)
- net LED_green: now reaches J3.18 (BCM24)
- net Input_SW3: now reaches J3.21 (BCM9)
- net LED_blue: now reaches J3.22 (BCM25)
- net Input_SW2: now reaches J3.29 (BCM5)
- net UC_Reset: now reaches J3.31 (BCM6)
- net Data_to_UC: now reaches J3.32 (BCM12)
- net Data_from_UC: now reaches J3.33 (BCM13)
- net Input_SW1: now reaches J3.7 (BCM4)
- net Console_TX: now reaches J3.8 (BCM14)
- new net: U5.10 (VCC), U5.31 (VCC), U5.61 (VCC), U5.80 (VCC)
- new net: U5.11 (GND), U5.32 (GND), U5.62 (GND), U5.81 (GND), U5.99 (GND)
- new net: U4.29 (GND), U4.3 (GND)
- new net +5V: C1.1, J3.2 (P5V), J3.4 (P5V)
Other:
- moved on the sheet: H1, H2, H3, H4, J6, J9, Q1, Q2A, Q2B, R11, R23, R24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
